Commit message: Some changes to the launch file and to the model.  Minor edits.

File: tdx_urdf/otto.xacro (robot description, xacro)
@@ -3,7 +3,7 @@
   <xacro:property name="pi" value="3.14159265358979" />
   <!-- The total size for the collision boudning box. -->
-  <xacro:property name="colllen" value="0.4318" />
-  <xacro:property name="collwidth" value="0.3302" />
-  <xacro:property name="collheight" value="0.254" />
+  <xacro:property name="colllen" value="1.14" />
+  <xacro:property name="collwidth" value="0.66" />
+  <xacro:property name="collheight" value="1.5" />
   <!-- The size of the battery box/area between the drive wheels. -->
   <xacro:property name="battlen" value="0.4318" />
@@ -27,5 +27,5 @@
       </geometry>
       <material name="collision">
-	<color rgba="1 0 0 0.2"/>
+	<color rgba="1 0 0 0.5"/>
       </material>
     </collision>

Commit message: Finished the Otto URDF.  Yay!

File: tdx_urdf/otto.xacro (robot description, xacro)
@@ -3,7 +3,10 @@
   <xacro:property name="pi" value="3.14159265358979" />
   <!-- The total size for the collision boudning box. -->
-  <xacro:property name="colllen" value="1.14" />
-  <xacro:property name="collwidth" value="0.66" />
-  <xacro:property name="collheight" value="1.5" />
+  <xacro:property name="colllen" value="1.08" />
+  <xacro:property name="collwidth" value="0.68" />
+  <xacro:property name="collheight" value="1.65" />
+  <xacro:property name="colloffsetx" value="0.141" />
+  <xacro:property name="colloffsety" value="0.0" />
+  <xacro:property name="colloffsetz" value="0.0" />
   <!-- The size of the battery box/area between the drive wheels. -->
   <xacro:property name="battlen" value="0.4318" />
@@ -22,12 +25,4 @@
       </material>
     </visual>
-    <collision>
-      <geometry>
-	<box size="${colllen} ${collwidth} ${collheight}"/>
-      </geometry>
-      <material name="collision">
-	<color rgba="1 0 0 0.5"/>
-      </material>
-    </collision>
   </link>
   <joint name="base_to_batt_box" type="fixed">
@@ -35,4 +30,41 @@
     <child link="battery_box"/>
     <origin xyz="0 0 ${battheight/2.0+0.04445}"/>
+  </joint>
+    <link name="collision_box">
+    <visual>
+      <geometry>
+	<box size="0.01 0.01 0.01"/>
+      </geometry>
+      <material name="collision">
+	<color rgba="0.8 0.8 1 0.1"/>
+      </material>
+    </visual>
+    <collision>
+      <geometry>
+	<box size="${colllen} ${collwidth} ${collheight}"/>
+      </geometry>
+      <origin xyz="${colloffsetx} ${colloffsety} ${colloffsetz+collheight/2.0-(battheight/2.0+0.04445)}"/>
+    </collision>
+  </link>
+  <joint name="batt_to_collision_box" type="fixed">
+    <parent link="battery_box"/>
+    <child link="collision_box"/>
+    <origin xyz="0 0 0"/>
+  </joint>
+  <!-- Main battery box -->
+  <link name="seat_lift">
+    <visual>
+      <geometry>
+	<box size="0.2 0.2 0.15"/>
+      </geometry>
+      <material name="black">
+	<color rgba="0 0 0 1"/>
+      </material>
+    </visual>
+  </link>
+  <joint name="batt_box_to_seat_lift" type="fixed">
+    <parent link="battery_box"/>
+    <child link="seat_lift"/>
+    <origin xyz="0 0 ${battheight/2.0-0.02}"/>
   </joint>
   <!-- Tires and drive motors -->
@@ -67,5 +99,5 @@
 	<origin xyz="0 0 0" rpy="0 0 0"/>
 	<material name="tire">
-	  <color rgba="0.65 0.65 0.6 1"/>
+	  <color rgba="0.45 0.45 0.47 1"/>
 	</material>
       </visual>
@@ -95,4 +127,159 @@
   <xacro:drivewheel prefix="right" reflect="-1" />
   <xacro:drivewheel prefix="left" reflect="1" />
+    <!-- Macro for the front casters -->
+  <xacro:property name="casterradius" value="0.0762" />
+  <xacro:property name="casterwidth" value="0.0381" />
+  <xacro:property name="casterhubradius" value="0.055" />
+  <xacro:property name="casterhubwidth" value="0.04" />
+  <xacro:property name="casterheight" value="0.15" />
+  <xacro:macro name="frontcaster" params="prefix reflect">
+    <link name="${prefix}_caster_leg">
+      <visual>
+	<geometry>
+	  <box size="0.04445 0.04445 ${casterheight}"/>
+	</geometry>
+	<origin xyz="0 0 0" rpy="0 0 0"/>
+	<material name="black">
+	  <color rgba="0 0 0 1"/>
+	</material>
+      </visual>
+    </link>
+    <link name="${prefix}_caster">
+      <visual>
+	<geometry>
+	  <cylinder length="${casterwidth}" radius="${casterradius}"/>
+	</geometry>
+	<material name="caster">
+	  <color rgba="0.3 0.3 0.26 1"/>
+	</material>
+      </visual>
+    </link>
+    <joint name="${prefix}_caster_leg_to_${prefix}_caster" type="fixed">
+      <parent link="${prefix}_caster_leg"/>
+      <child link="${prefix}_caster"/>
+      <origin xyz="0 0 -0.03" rpy="${pi/2} 0 0"/>
+    </joint>
+    <link name="${prefix}_caster_hub">
+      <visual>
+	<geometry>
+	  <cylinder length="${casterhubwidth}" radius="${casterhubradius}"/>
+	</geometry>
+	<material name="black">
+	  <color rgba="0 0 0 1"/>
+	</material>
+      </visual>
+    </link>
+    <joint name="${prefix}_caster_hub_to_${prefix}_caster" type="fixed">
+      <parent link="${prefix}_caster"/>
+      <child link="${prefix}_caster_hub"/>
+      <origin xyz="0 0 0" rpy="0 0 0"/>
+    </joint>
+    <link name="${prefix}_caster_bar_aux">
+      <visual>
+	<geometry>
+	  <cylinder length="0.20" radius="0.02"/>
+	</geometry>
+	<origin xyz="0 0 0" rpy="0 ${pi/2} 0"/>
+	<material name="silver">
+	  <color rgba="0.4 0.4 0.4 1"/>
+	</material>
+      </visual>
+    </link>
+    <joint name="${prefix}_caster_bar_aux_joint" type="fixed">
+      <parent link="${prefix}_caster_bar"/>
+      <child link="${prefix}_caster_bar_aux"/>
+      <origin xyz="0.10 ${reflect*-0.02} -0.05" rpy="0 -0.6 ${reflect*0.3}"/>
+    </joint>
+    <link name="${prefix}_caster_bar">
+      <visual>
+	<geometry>
+	  <cylinder length="0.38" radius="0.02"/>
+	</geometry>
+	<origin xyz="0 0 0" rpy="0 ${pi/2} 0"/>
+	<material name="silver">
+	  <color rgba="0.4 0.4 0.4 1"/>
+	</material>
+      </visual>
+    </link>
+    <joint name="${prefix}_caster_bar_joint" type="fixed">
+      <parent link="${prefix}_caster_bar"/>
+      <child link="${prefix}_caster_leg"/>
+      <origin xyz="0.16 0 ${-casterradius}" rpy="0 -0.2 ${reflect*(pi-0.1)}"/>
+    </joint>
+    <joint name="${prefix}_to_caster" type="fixed">
+      <parent link="battery_box"/>
+      <child link="${prefix}_caster_bar"/>
+      <origin xyz="0.18 ${reflect*(battwidth/2.0+0.05)} 0.05" rpy="0 0.3 ${reflect*0.1}"/>
+    </joint>
+  </xacro:macro>
+  <xacro:frontcaster prefix="front_right" reflect="-1" />
+  <xacro:frontcaster prefix="front_left" reflect="1" />
+  <!-- Macro for the rear casters -->
+  <xacro:macro name="rearcaster" params="prefix reflect">
+    <link name="${prefix}_caster_leg">
+      <visual>
+	<geometry>
+	  <box size="0.04445 0.04445 ${casterheight}"/>
+	</geometry>
+	<origin xyz="0 0 0" rpy="0 0 0"/>
+	<material name="black">
+	  <color rgba="0 0 0 1"/>
+	</material>
+      </visual>
+    </link>
+    <link name="${prefix}_caster">
+      <visual>
+	<geometry>
+	  <cylinder length="${casterwidth}" radius="${casterradius}"/>
+	</geometry>
+	<material name="caster">
+	  <color rgba="0.3 0.3 0.26 1"/>
+	</material>
+      </visual>
+    </link>
+    <joint name="${prefix}_caster_leg_to_${prefix}_caster" type="fixed">
+      <parent link="${prefix}_caster_leg"/>
+      <child link="${prefix}_caster"/>
+      <origin xyz="0 0 -0.03" rpy="${pi/2} 0 0"/>
+    </joint>
+    <link name="${prefix}_caster_hub">
+      <visual>
+	<geometry>
+	  <cylinder length="${casterhubwidth}" radius="${casterhubradius}"/>
+	</geometry>
+	<material name="black">
+	  <color rgba="0 0 0 1"/>
+	</material>
+      </visual>
+    </link>
+    <joint name="${prefix}_caster_hub_to_${prefix}_caster" type="fixed">
+      <parent link="${prefix}_caster"/>
+      <child link="${prefix}_caster_hub"/>
+      <origin xyz="0 0 0" rpy="0 0 0"/>
+    </joint>
+    <link name="${prefix}_caster_bar">
+      <visual>
+	<geometry>
+	  <cylinder length="0.1524" radius="0.02"/>
+	</geometry>
+	<origin xyz="0 0 0" rpy="0 ${pi/2.0} 0"/>
+	<material name="silver">
+	  <color rgba="0.4 0.4 0.4 1"/>
+	</material>
+      </visual>
+    </link>
+    <joint name="${prefix}_caster_bar_joint" type="fixed">
+      <parent link="${prefix}_caster_bar"/>
+      <child link="${prefix}_caster_leg"/>
+      <origin xyz="-0.0712 0 ${-casterradius}" rpy="0 -0.2 ${pi}"/>
+    </joint>
+    <joint name="${prefix}_to_caster" type="fixed">
+      <parent link="battery_box"/>
+      <child link="${prefix}_caster_bar"/>
+      <origin xyz="${-battlen/2.0-0.0712/2.0} ${reflect*0.12} 0" rpy="0 0 0"/>
+    </joint>
+  </xacro:macro>
+  <xacro:rearcaster prefix="back_right" reflect="-1" />
+  <xacro:rearcaster prefix="back_left" reflect="1" />
   <!-- Rider Cushion -->
   <xacro:property name="seatlen" value="0.4445" />
@@ -104,6 +291,6 @@
 	<box size="${seatlen} ${seatwidth} ${seatheight}"/>
       </geometry>
-      <material name="black">
-	<color rgba="0 0 0 1"/>
+      <material name="lightblack">
+	<color rgba="0.025 0.025 0.04 1"/>
       </material>
     </visual>
@@ -113,4 +300,112 @@
     <child link="rider_seat"/>
     <origin xyz="0.13 0 0.2"/>
+  </joint>
+  <!-- Armrests -->
+  <xacro:property name="armrestpolelen" value="0.18" />
+  <xacro:property name="armrestpoleradius" value="0.01" />
+  <xacro:property name="armrestwidth" value="0.0635" />
+  <xacro:property name="armrestthickness" value="0.04" />
+  <xacro:macro name="armrest" params="prefix armrestlength poleseparation">
+    <link name="${prefix}_front_armrest_pole">
+      <visual>
+	<geometry>
+	  <cylinder length="${armrestpolelen}" radius="${armrestpoleradius}"/>
+	</geometry>
+	<origin xyz="0 0 0" rpy="0 0 0"/>
+	<material name="black">
+	  <color rgba="0 0 0 1"/>
+	</material>
+      </visual>
+    </link>
+    <link name="${prefix}_rear_armrest_pole">
+      <visual>
+	<geometry>
+	  <cylinder length="${armrestpolelen}" radius="${armrestpoleradius}"/>
+	</geometry>
+	<origin xyz="0 0 0" rpy="0 0 0"/>
+	<material name="black">
+	  <color rgba="0 0 0 1"/>
+	</material>
+      </visual>
+    </link>
+    <joint name="${prefix}_armrest_pole_to_pole" type="fixed">
+      <parent link="${prefix}_front_armrest_pole"/>
+      <child link="${prefix}_rear_armrest_pole"/>
+      <origin xyz="${-poleseparation} 0 0" rpy="0 0 0"/>
+    </joint>
+    <link name="${prefix}_armrest_pad">
+      <visual>
+	<geometry>
+	  <box size="${armrestlength} ${armrestwidth} ${armrestthickness}"/>
+	</geometry>
+      <material name="lightblack">
+	<color rgba="0.025 0.025 0.04 1"/>
+      </material>
+      </visual>
+    </link>
+  <joint name="${prefix}_armrest_pad_to_pole" type="fixed">
+    <parent link="${prefix}_front_armrest_pole"/>
+    <child link="${prefix}_armrest_pad"/>
+    <origin xyz="${-0.25*armrestlength} 0 ${armrestpolelen/2.0}"/>
+  </joint>
+  </xacro:macro>
+  <xacro:property name="rightarmrestlength" value="0.3048" />
+  <xacro:armrest prefix="left" armrestlength="0.4318" poleseparation="0.3048" />
+  <xacro:armrest prefix="right" armrestlength="${rightarmrestlength}" poleseparation="0.20" />
+  <joint name="seat_to_left_armrest" type="fixed">
+    <parent link="rider_seat"/>
+    <child link="left_front_armrest_pole"/>
+    <origin xyz="0.13 ${seatwidth/2.0} ${armrestpolelen/2.0}"/>
+  </joint>
+  <joint name="seat_to_right_armrest" type="fixed">
+    <parent link="rider_seat"/>
+    <child link="right_front_armrest_pole"/>
+    <origin xyz="0 ${-seatwidth/2.0} ${armrestpolelen/2.0}"/>
+  </joint>
+  <!-- Control Joystick -->
+  <link name="joystick_box">
+    <visual>
+      <geometry>
+	<box size="0.1778 0.0635 0.0508"/>
+      </geometry>
+      <material name="black">
+	<color rgba="0 0 0 1"/>
+      </material>
+    </visual>
+  </link>
+  <joint name="right_armrest_to_joystick_box" type="fixed">
+    <parent link="right_armrest_pad"/>
+    <child link="joystick_box"/>
+    <origin xyz="${rightarmrestlength/2.0+0.105} -0.01 0"/>
+  </joint>
+  <link name="joystick_ball">
+    <visual>
+      <geometry>
+	<sphere radius="0.01651"/>
+      </geometry>
+      <material name="lightblack">
+	<color rgba="0.025 0.025 0.04 1"/>
+      </material>
+    </visual>
+  </link>
+  <joint name="joystick_box_to_ball" type="fixed">
+    <parent link="joystick_box"/>
+    <child link="joystick_ball"/>
+    <origin xyz="0.04 0 0.03175"/>
+  </joint>
+  <link name="joystick_stick">
+    <visual>
+      <geometry>
+	<cylinder length="0.05" radius="0.007"/>
+      </geometry>
+      <material name="lightblack">
+	<color rgba="0.025 0.025 0.04 1"/>
+      </material>
+    </visual>
+  </link>
+  <joint name="joystick_ball_to_stick" type="fixed">
+    <parent link="joystick_ball"/>
+    <child link="joystick_stick"/>
+    <origin xyz="0 0 0.009525"/>
   </joint>
   <!-- Rider Back -->
@@ -133,59 +428,4 @@
     <origin xyz="-0.18 0 0.4"/>
   </joint>
-  <!-- Macro for the rear casters -->
-  <xacro:property name="casterradius" value="0.0762" />
-  <xacro:property name="casterwidth" value="0.0381" />
-  <xacro:property name="casterheight" value="0.15" />
-  <xacro:macro name="rearcaster" params="prefix reflect">
-    <link name="${prefix}_caster_leg">
-      <visual>
-	<geometry>
-	  <box size="0.04445 0.04445 ${casterheight}"/>
-	</geometry>
-	<origin xyz="0 0 0" rpy="0 0 0"/>
-	<material name="black">
-	  <color rgba="0 0 0 1"/>
-	</material>
-      </visual>
-    </link>
-    <link name="${prefix}_caster">
-      <visual>
-	<geometry>
-	  <cylinder length="${casterwidth}" radius="${casterradius}"/>
-	</geometry>
-	<material name="caster">
-	  <color rgba="0.55 0.55 0.44 1"/>
-	</material>
-      </visual>
-    </link>
-    <joint name="${prefix}_caster_leg_to_${prefix}_caster" type="fixed">
-      <parent link="${prefix}_caster_leg"/>
-      <child link="${prefix}_caster"/>
-      <origin xyz="0 0 -0.03" rpy="${pi/2} 0 0"/>
-    </joint>
-    <link name="${prefix}_caster_bar">
-      <visual>
-	<geometry>
-	  <cylinder length="0.1524" radius="0.02"/>
-	</geometry>
-	<origin xyz="0 0 0" rpy="0 ${pi/2.0} 0"/>
-	<material name="silver">
-	  <color rgba="0.3 0.3 0.35 1"/>
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